Commit message: Lidar Pose update

File: myRobot_ws/src/myrobot/urdf/myrobot.urdf.xacro (robot description, xacro)
@@ -844,5 +844,5 @@
   <link name="lidar_link">
     <visual>
-      <origin xyz="0.0 0 0.073" rpy="0 0 0"/>
+      <origin xyz="0.0 0 0.0" rpy="0 0 0"/>
       <geometry>
         <mesh
@@ -851,5 +851,5 @@
     </visual>
     <collision>
-      <origin xyz="0.0 0 0.073" rpy="0 0 0"/>
+      <origin xyz="0.0 0 0.0" rpy="0 0 0"/>
       <geometry>
         <mesh
@@ -858,5 +858,5 @@
     </collision>
     <inertial>
-      <origin xyz="0.0 0 0.073" rpy="0 0 0"/>
+      <origin xyz="0.0 0 0.0" rpy="0 0 0"/>
       <mass value="1"/>
       <inertia ixx="0.1" ixy="0" ixz="0" iyy="0.1" iyz="0" izz="0.1"/>
@@ -865,5 +865,5 @@
   <!-- Define joint connecting base link and LiDAR link -->
   <joint name="lidar_joint" type="fixed">
-    <origin xyz="0 0 0" rpy="0 0 0"/>
+    <origin xyz="0 0 0.073" rpy="0 0 3.14"/>
     <parent link="base_link"/>
     <child link="lidar_link"/>
@@ -871,5 +871,5 @@
 <gazebo reference="lidar_link">
   <sensor name="lidar" type="ray">
-    <pose>0.0 0.0 0.08 0 0 3.14</pose>
+    <!-- <pose>0.0 0.0 0.08 0 0 3.14</pose> -->
     <always_on>true</always_on>
     <visualize>true</visualize>
